Commit message: Agregar garra paralela de dos dedos al robot

File: HandRecognition/hachi.urdf (robot description, URDF)
Before this commit: robot humanoid_shoulder_arm_l_shape, 7 links, 6 joints
Links:
- removed link gripper_link
- added link gripper_base_link, mass 0.20; collision box size=0.08 0.08 0.05; visual box size=0.08 0.08 0.05
- added link left_finger_link, mass 0.08; collision box size=0.025 0.025 0.12; visual box size=0.025 0.025 0.12
- added link right_finger_link, mass 0.08; collision box size=0.025 0.025 0.12; visual box size=0.025 0.025 0.12
Joints:
- added joint gripper_base_joint: type fixed, parent wrist_2_link, child gripper_base_link, origin xyz=0 0 -0.10 rpy=0 0 0
- added joint joint_7: type prismatic, parent gripper_base_link, child right_finger_link, origin xyz=0 -0.015 -0.05 rpy=0 0 0, axis 0 1 0, limit lower=-0.04 upper=0.0 effort=10 velocity=0.20
- joint joint_6: axis 1 0 0 -> 0 1 0; child gripper_link -> left_finger_link; limit lower=0.0 upper=0.8 effort=10 velocity=5.0 -> lower=0.0 upper=0.04 effort=10 velocity=0.20; origin xyz=0 0 -0.1 rpy=0 0 0 -> xyz=0 0.015 -0.05 rpy=0 0 0; parent wrist_2_link -> gripper_base_link; type revolute -> prismatic
